File: Eagle Files/GPSPassive.sch (EAGLE design)
At the start: 57 parts, among them SW1 SPST_TACT-KMR2, SW2 KMR2, SW3 KMR2, U1 ATSAMD21G-A, U2 SPX3819-3.3, U3 MCP73831T-2ACI/OT, X1 JSTPH, X2 uFL, X3 microUSB, X4 uFL, X5 uFL, X6 SIM_LOCKAMPHENOL, Y1 32.768kHz

Commit message: Agrega board principal
Parts:
- added C18, C19, C20: 1uF, microbuilder:CAP_CERAMIC0805-NOOUTLINE
- added D11: RED, microbuilder:LED0805_NOOUTLINE
- added D12: GREEN, microbuilder:LED0805_NOOUTLINE
- added J2: (no value), SparkFun-Connectors:M05X2SHD_LOCK
- added R12, R13: 1K, microbuilder:RESISTOR0805_NOOUTLINE
- added U$1: MICROSD, adafruit:MICROSD
- added U5: (no value), microbuilder:NRF51822_MODULE_MDBT40
- added Y2: 32.768kHz (535-9166-2-ND), microbuilder:CRYSTAL2.0X6.0_32.768
Connections:
- new net CONNECTED_LED: R13.1, U5.P0.19
- new net MISO: U$1.DATA_OUT, U1.PA19(SER1:3+)
- new net MODE_LED: R12.1, U5.P0.18
- new net MOSI: U$1.DATA_IN, U1.PA16(I2C/SER1:0+)
- new net N$26: D11.A, R12.2
- new net N$27: D12.A, R13.2
- new net N$28: C19.1, U5.P0.26/AIN0/XL2, Y2.1
- new net N$29: C20.1, U5.P0.27/AIN1/XL1, Y2.2
- new net N$30: C18.1, J2.4, U5.AVDD, U5.VDD
- new net N$31: J2.1, U5.SWCLK
- new net N$32: J2.5, J2.6, U5.SWDIO/NRESET
- new net RX_BT: U1.PA10(AIN18/SER0:2+), U5.P0.11
- new net SCK: U$1.SCLK, U1.PA17(I2C/SER1:1+)
- new net SD_CS: U$1.CS, U1.PB08(AIN2/SER4:0/TC4:0)
- new net TX_BT: U1.PA11(AIN19/SER0:3+), U5.P0.09
- net GND: now also C18.2, C19.2, C20.2, D11.C, D12.C, J2.2, U$1.GND, U5.GND@1, U5.GND@2, U5.GND@3, U5.GND@4, U5.GND@5, U5.P0.30
- net N$2: now also U1.PA00(XIN32/SER1:0/TC2:0)
- net N$4: now also U1.PA01(XOUT32/SER1:1/TC2:1)
- net VCC: now also U$1.VDD
Other:
- moved on the sheet: X6

Commit message: Corrige colocación de LED
Parts:
- removed PWRSTAT: RED, microbuilder:LED0805_NOOUTLINE
- removed R5, R9: 1K, microbuilder:RESISTOR0805_NOOUTLINE
- removed U2: SPX3819-3.3, microbuilder:VREG_SOT23-5
- added AP2114H: REG1117, burr-brown:REG1117
- added PWR: RED, microbuilder:LED0805_NOOUTLINE
- added R14: 1K, microbuilder:RESISTOR0805_NOOUTLINE
- J1, J2: device SparkFun-Connectors:M05X2SHD_LOCK -> SparkFun-Connectors:M05PTH
- R1: value 100k -> 1K; device microbuilder:RESISTOR_0603_NOOUT -> microbuilder:RESISTOR0805_NOOUTLINE
- R8: value 10K\ -> 1K
- renumbered D11 to MODE, D12 to CONN, NETSTAT to NETLIGHT
Connections:
- removed net EN: R1.2, U2.EN
- removed net N$21: PWRSTAT.A, R5.1
- removed net N$30: C18.1, J2.4, U5.AVDD, U5.VDD
- new net N$33: PWR.A, R14.1
- net !RESET: now also J1.2; no longer J1.6
- net GND: now also AP2114H.GND, J1.3, J2.3, PWR.C; no longer J1.2, J2.2, PWRSTAT.C, U2.GND
- net N$14: now also AP2114H.VIN; no longer R1.1, U2.IN
- net N$20: now also R1.1; no longer R9.1
- net N$3: now also J1.4; no longer J1.1
- net N$31: now also J2.4; no longer J2.1
- net N$32: no longer J2.6
- net N$5: no longer J1.3
- net NS_P: now also R1.2; no longer R9.2
- net PS_P: no longer R5.2
- net VCC: now also AP2114H.VOUT, C18.1, J1.1, J2.1, R14.2, U5.AVDD, U5.VDD; no longer J1.4, U2.OUT
Other:
- moved on the sheet: R1

Commit message: Corrige inversión de pines TX y RX para BLE
Parts:
- removed AP2114H: REG1117, burr-brown:REG1117
- removed PWR: RED, microbuilder:LED0805_NOOUTLINE
- removed R14: 1K, microbuilder:RESISTOR0805_NOOUTLINE
- added PWRSTAT: RED, microbuilder:LED0805_NOOUTLINE
- added R5, R9: 1K, microbuilder:RESISTOR0805_NOOUTLINE
- added U2: SPX3819-3.3, microbuilder:VREG_SOT23-5
- J1, J2: device SparkFun-Connectors:M05PTH -> SparkFun-Connectors:M05X2SHD_LOCK
- R1: value 1K -> 100k; device microbuilder:RESISTOR0805_NOOUTLINE -> microbuilder:RESISTOR_0603_NOOUT
- R8: value 1K -> 10K\
- renumbered CONN to D12, MODE to D11, NETLIGHT to NETSTAT
Connections:
- removed net N$33: PWR.A, R14.1
- new net EN: R1.2, U2.EN
- new net N$21: PWRSTAT.A, R5.1
- new net N$30: C18.1, J2.4, U5.AVDD, U5.VDD
- net !RESET: now also J1.6; no longer J1.2
- net GND: now also J1.2, J2.2, PWRSTAT.C, U2.GND; no longer AP2114H.GND, J1.3, J2.3, PWR.C
- net N$14: now also R1.1, U2.IN; no longer AP2114H.VIN
- net N$20: now also R9.1; no longer R1.1
- net N$3: now also J1.1; no longer J1.4
- net N$31: now also J2.1; no longer J2.4
- net N$32: now also J2.6
- net N$5: now also J1.3
- net NS_P: now also R9.2; no longer R1.2
- net PS_P: now also R5.2
- net VCC: now also J1.4, U2.OUT; no longer AP2114H.VOUT, C18.1, J1.1, J2.1, R14.2, U5.AVDD, U5.VDD
Other:
- moved on the sheet: R1
